File: hi-amp-pwm/MAN-PWM-CTR.kicad_pcb (KiCad board)
At the start: 2 copper layers, 16 parts, among them J1 TRM-RHE, J2 PWR/PWM, Q1 Q_NMOS_GDS, U1 NE555, U2 NE555

Commit message: Addded ReadMe.txt files to aid use, and deleted missed backup files
Parts:
- Q1: value Q_NMOS_GDS -> IRF540
Other:
- net class Default removed
